Commit message: added two wheels

File: urdf/my_robot.xacro (robot description, xacro)
@@ -6,4 +6,44 @@
     <parent link="robot_footprint"/>
     <child link="chassis" />
+  </joint>
+	<link name='left_wheel'>
+		<geometry>
+			<cylinder radius="0.1" length="0.05"/>
+		</geometry>
+		<origin xyz="0 0 0" rpy="0 1.5701 1.5707"/>
+		<mass value="5"/>
+		<inertia
+    	ixx="0.1" ixy="0" ixz="0"
+      iyy="0.1" iyz="0"
+      izz="0.1"
+		/>
+	</link>
+	<link name='right_wheel'>
+		<geometry>
+			<cylinder radius="0.1" length="0.05"/>
+		</geometry>
+		<origin xyz="0 0 0" rpy="0 1.5701 1.5707"/>
+		<mass value="5"/>
+		<inertia
+    	ixx="0.1" ixy="0" ixz="0"
+      iyy="0.1" iyz="0"
+      izz="0.1"
+		/>
+	</link>
+  <joint type="continuous" name="left_wheel_hinge">
+    <origin xyz="0 0.15 0" rpy="0 0 0"/>
+    <child link="left_wheel"/>
+    <parent link="chassis"/>
+    <axis xyz="0 1 0" rpy="0 0 0"/>
+    <limit effort="10000" velocity="1000"/>
+    <dynamics damping="1.0" friction="1.0"/>
+  </joint>
+  <joint type="continuous" name="right_wheel_hinge">
+    <origin xyz="0 0.15 0" rpy="0 0 0"/>
+    <child link="right_wheel"/>
+    <parent link="chassis"/>
+    <axis xyz="0 1 0" rpy="0 0 0"/>
+    <limit effort="10000" velocity="1000"/>
+    <dynamics damping="1.0" friction="1.0"/>
   </joint>
   <link name='chassis'>

Commit message: updated joins for wheels

File: urdf/my_robot.xacro (robot description, xacro)
@@ -8,26 +8,48 @@
   </joint>
 	<link name='left_wheel'>
-		<geometry>
-			<cylinder radius="0.1" length="0.05"/>
-		</geometry>
-		<origin xyz="0 0 0" rpy="0 1.5701 1.5707"/>
-		<mass value="5"/>
-		<inertia
-    	ixx="0.1" ixy="0" ixz="0"
-      iyy="0.1" iyz="0"
-      izz="0.1"
-		/>
+		<inertial>
+      <mass value="5"/>
+      <origin xyz="0 0 0" rpy="0 1.5701 1.5707"/>
+      <inertia
+          ixx="0.1" ixy="0" ixz="0"
+          iyy="0.1" iyz="0"
+          izz="0.1"
+      />
+    </inertial>
+    <collision name='collision'>
+      <origin xyz="0 0 0" rpy="0 1.5701 1.5707"/>
+			<geometry>
+				<cylinder radius="0.1" length="0.05"/>
+			</geometry>
+    </collision>
+    <visual name='left_wheel_visual'>
+      <origin xyz="0 0 0" rpy="0 1.5701 1.5707"/>
+			<geometry>
+				<cylinder radius="0.1" length="0.05"/>
+			</geometry>
+    </visual>
 	</link>
 	<link name='right_wheel'>
-		<geometry>
-			<cylinder radius="0.1" length="0.05"/>
-		</geometry>
-		<origin xyz="0 0 0" rpy="0 1.5701 1.5707"/>
-		<mass value="5"/>
-		<inertia
-    	ixx="0.1" ixy="0" ixz="0"
-      iyy="0.1" iyz="0"
-      izz="0.1"
-		/>
+		<inertial>
+      <mass value="5"/>
+      <origin xyz="0 0 0" rpy="0 1.5701 1.5707"/>
+      <inertia
+          ixx="0.1" ixy="0" ixz="0"
+          iyy="0.1" iyz="0"
+          izz="0.1"
+      />
+    </inertial>
+    <collision name='collision'>
+      <origin xyz="0 0 0" rpy="0 1.5701 1.5707"/>
+			<geometry>
+				<cylinder radius="0.1" length="0.05"/>
+			</geometry>
+    </collision>
+    <visual name='right_wheel_visual'>
+      <origin xyz="0 0 0" rpy="0 1.5701 1.5707"/>
+			<geometry>
+				<cylinder radius="0.1" length="0.05"/>
+			</geometry>
+    </visual>
 	</link>
   <joint type="continuous" name="left_wheel_hinge">
@@ -40,5 +62,5 @@
   </joint>
   <joint type="continuous" name="right_wheel_hinge">
-    <origin xyz="0 0.15 0" rpy="0 0 0"/>
+    <origin xyz="0 -0.15 0" rpy="0 0 0"/>
     <child link="right_wheel"/>
     <parent link="chassis"/>

Commit message: updated joins for wheels

File: urdf/my_robot.xacro (robot description, xacro)
@@ -117,3 +117,26 @@
     </visual>
   </link>
+	<link name="camera">
+		<inertial>
+      <mass value=".1"/>
+      <origin xyz="0 0 0" rpy="0 0 0"/>
+      <inertia
+          ixx="1e-6" ixy="0" ixz="0"
+          iyy="1e-6" iyz="0"
+          izz="1e-6"
+      />
+    </inertial>
+    <collision name='collision'>
+      <origin xyz="0 0 0" rpy="0 0 0"/>
+      <geometry>
+        <box size=".05 .05 .05"/>
+      </geometry>
+    </collision>
+    <visual name='camera_visual'>
+      <origin xyz="0 0 0" rpy=" 0 0 0"/>
+      <geometry>
+        <box size=".05 .05 .05"/>
+      </geometry>
+    </visual>
+	</link>
 </robot>

Commit message: added camera sencor

File: urdf/my_robot.xacro (robot description, xacro)
@@ -126,4 +126,5 @@
           izz="1e-6"
       />
+			<box_inertia m="0.1" x="0.05" y="0.05" z="0.05"/>
     </inertial>
     <collision name='collision'>
@@ -140,3 +141,9 @@
     </visual>
 	</link>
+  <joint type="fixed" name="camera_joint">
+    <origin xyz="0.2 0 0" rpy="0 0 0"/>
+    <child link="camera"/>
+    <parent link="chassis"/>
+    <axis xyz="0 1 0" rpy="0 0 0"/>
+  </joint>
 </robot>

Commit message: added lidar

File: urdf/my_robot.xacro (robot description, xacro)
@@ -147,3 +147,35 @@
     <axis xyz="0 1 0" rpy="0 0 0"/>
   </joint>
+  <link name="hokuyo">
+		<inertial>
+      <mass value="1e-5"/>
+      <origin xyz="0 0 0" rpy="0 0 0"/>
+      <inertia
+          ixx="1e-6" ixy="0" ixz="0"
+          iyy="1e-6" iyz="0"
+          izz="1e-6"
+      />
+    </inertial>
+    <collision name='collision'>
+      <origin xyz="0 0 0" rpy="0 0 0"/>
+      <geometry>
+        <box size=".1 .1 .1"/>
+      </geometry>
+    </collision>
+    <visual name='hokuyo_visual'>
+      <origin xyz="0 0 0" rpy=" 0 0 0"/>
+      <geometry>
+        <mesh filename="package://mybot_description/meshes/hokuyo.dae"/>
+      </geometry>
+    </visual>
+	</link>
+  <joint type="fixed" name="hokuyo_joint">
+    <origin xyz="0.15 0 .1" rpy="0 0 0"/>
+    <child link="hokuyo"/>
+    <parent link="chassis"/>
+    <axis xyz="0 1 0" rpy="0 0 0"/>
+  </joint>
+  <gazebo reference="chassis">
+      <material>Gazebo/Blue</material>
+  </gazebo>
 </robot>

Commit message: fixed file name of lidar

File: urdf/my_robot.xacro (robot description, xacro)
@@ -166,5 +166,5 @@
       <origin xyz="0 0 0" rpy=" 0 0 0"/>
       <geometry>
-        <mesh filename="package://mybot_description/meshes/hokuyo.dae"/>
+        <mesh filename="package:/my_robot/meshes/hokuyo.dae"/>
       </geometry>
     </visual>

Commit message: added colors to elements

File: urdf/my_robot.xacro (robot description, xacro)
@@ -166,5 +166,5 @@
       <origin xyz="0 0 0" rpy=" 0 0 0"/>
       <geometry>
-        <mesh filename="package:/my_robot/meshes/hokuyo.dae"/>
+        <mesh filename="package://my_robot/meshes/hokuyo.dae"/>
       </geometry>
     </visual>
@@ -179,3 +179,9 @@
       <material>Gazebo/Blue</material>
   </gazebo>
+  <gazebo reference="hokuyo">
+      <material>Gazebo/Black</material>
+  </gazebo>
+  <gazebo reference="camera">
+      <material>Gazebo/Red</material>
+  </gazebo>
 </robot>
